File: BLDC_driver.kicad_sch (KiCad schematic)
At the start: 0 parts

Commit message: Schematic complete
Completed power and controller sub-schematics, ESD protection

Not completed: componenet values and footprints

Not started: PCB layout design
Other:
- title: (none) -> Main schematic
Changed lines of the file:
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@@
 	(generator_version "8.0")
 	(paper "A4")
+	(title_block
+		(title "Main schematic")
+	)
 	(sheet
 		(at 161.29 62.23)
