File: power.kicad_sch (KiCad schematic)
At the start: 0 parts

Commit message: Schematic complete
Completed power and controller sub-schematics, ESD protection

Not completed: componenet values and footprints

Not started: PCB layout design
Parts:
- added C6: 10u, symbol Device:C
- added R4: 0, symbol Device:R
- added TP4: V+, symbol Connector:TestPoint
- added TP5: GND, symbol Connector:TestPoint
Connections:
- new net GND: R4.2
- new net GNDPWR: C6.2, R4.1, TP5.1
- new net VDD: C6.1, TP4.1
Other:
- title: (none) -> Power

Commit message: PCB v1 complete
with images, README extended...
Parts:
- C6: footprint (none) -> Capacitor_SMD:C_0603_1608Metric
- R4: footprint (none) -> Resistor_SMD:R_0603_1608Metric
- TP4, TP5: footprint (none) -> TestPoint:TestPoint_Pad_3.0x3.0mm
Changed lines of the file:
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@@
 			)
 		)
-		(property "Footprint" ""
+		(property "Footprint" "TestPoint:TestPoint_Pad_3.0x3.0mm"
 			(at 109.22 91.44 0)
 			(effects
@@
 			)
 		)
-		(property "Footprint" ""
+		(property "Footprint" "Resistor_SMD:R_0603_1608Metric"
 			(at 135.89 98.298 90)
 			(effects
@@
 			)
 		)
-		(property "Footprint" ""
+		(property "Footprint" "Capacitor_SMD:C_0603_1608Metric"
 			(at 121.6152 86.36 0)
 			(effects
@@
 			)
 		)
-		(property "Footprint" ""
+		(property "Footprint" "TestPoint:TestPoint_Pad_3.0x3.0mm"
 			(at 109.22 66.04 0)
 			(effects

Commit message: C6 capacitor reviewed
Parts:
- C6: footprint Capacitor_SMD:C_0603_1608Metric -> Capacitor_SMD:C_0805_2012Metric
Changed lines of the file:
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@@
 			)
 		)
-		(property "Footprint" "Capacitor_SMD:C_0603_1608Metric"
+		(property "Footprint" "Capacitor_SMD:C_0805_2012Metric"
 			(at 121.6152 86.36 0)
 			(effects
